Commit message: test1 gravity rotation ok

File: src/bullet/rob1/arm2.urdf (robot description, URDF)
Before this commit: robot simple_arm, 4 links, 3 joints
Links:
- link arm1: mass None -> 2
- link arm2: mass None -> 2
- link wheel: mass None -> .1
Joints:
- joint joint3: limit lower=-1.57 upper=1.57 effort=1000 velocity=1.0 -> lower=-3.14 upper=3.14 effort=100 velocity=1.0

Commit message: update

File: src/bullet/rob1/arm2.urdf (robot description, URDF)
Before this commit: robot simple_arm, 4 links, 3 joints
Links:
- link arm1: geometry collision box size=0.1 0.1 2; visual box size=0.1 0.1 2
- link arm2: geometry collision box size=0.1 0.1 2; visual box size=0.1 0.1 2
- link arm3: geometry collision box size=0.1 0.1 2; visual box size=0.1 0.1 2
- link wheel: mass .1 -> 0; geometry collision cylinder length=0.1 radius=.25; visual cylinder length=0.1 radius=.25
Joints:
- joint joint2: limit lower=-1.57 upper=1.57 effort=1000 velocity=1 -> lower=-3.14 upper=3.14 effort=1000 velocity=1
- joint joint3: limit lower=-3.14 upper=3.14 effort=100 velocity=1.0 -> (none); type revolute -> continuous
