Commit message: test1 gravity rotation ok

File: src/bullet/rob1/test1.urdf (robot description, URDF)
Before this commit: robot simple_arm, 2 links, 1 joints
Links:
- link arm: geometry collision cylinder length=1 radius=0.1; visual cylinder length=1 radius=0.1
- link base: geometry collision cylinder length=1 radius=0.1; visual cylinder length=1 radius=0.1

Commit message: test with arm and hand

File: src/bullet/rob1/test1.urdf (robot description, URDF)
Before this commit: robot simple_arm, 2 links, 1 joints
Links:
- added link hand, mass 10; collision cylinder length=.4 radius=0.1; visual cylinder length=.4 radius=0.06
Joints:
- added joint joint1: type continuous, parent base, child arm, origin xyz=0 0 1 rpy=0 1.57 0, axis 0 1 0
- joint joint2: child arm -> hand; origin xyz=0 0 1 rpy=0 1.57 0 -> xyz=0 0 1 rpy=0 1 0; parent base -> arm

Commit message: simple gui

File: src/bullet/rob1/test1.urdf (robot description, URDF)
Before this commit: robot simple_arm, 3 links, 2 joints
Joints:
- joint joint2: origin xyz=0 0 1 rpy=0 1 0 -> xyz=0 0 1 rpy=0 -1.57 0
